Commit message: fix

File: config/minicar_diff_real.xacro (robot description, xacro)
@@ -1,6 +1,26 @@
 <?xml version="1.0"?>
 <robot name="minicar_diff_real" xmlns:xacro="http://www.ros.org/wiki/xacro">
-  <!-- Include base URDF -->
-  <xacro:include filename="$(find minicar_project)/robot_description/urdf/minicar_diff_gazebo.xacro" />
+  <!-- Minimal robot structure for hardware interface -->
+  <link name="base_link"/>
+  <link name="left_front_wheel"/>
+  <link name="right_front_wheel"/>
+  <link name="left_rear_wheel"/>
+  <link name="right_rear_wheel"/>
+  <joint name="left_front_wheel_joint" type="continuous">
+    <parent link="base_link"/>
+    <child link="left_front_wheel"/>
+  </joint>
+  <joint name="right_front_wheel_joint" type="continuous">
+    <parent link="base_link"/>
+    <child link="right_front_wheel"/>
+  </joint>
+  <joint name="left_rear_wheel_joint" type="continuous">
+    <parent link="base_link"/>
+    <child link="left_rear_wheel"/>
+  </joint>
+  <joint name="right_rear_wheel_joint" type="continuous">
+    <parent link="base_link"/>
+    <child link="right_rear_wheel"/>
+  </joint>
   <!-- Real hardware interface (replace Gazebo plugin) -->
   <ros2_control name="RealSystem" type="system">
@@ -9,8 +29,12 @@
       <param name="wheel_radius">0.035</param>
       <param name="encoder_ticks_per_revolution">1024</param>
-      <!-- I2C/PCA9685 configuration -->
       <param name="i2c_device">/dev/i2c-1</param>
       <param name="pca9685_address">64</param>
     </hardware>
+    <!--
+    <hardware>
+      <plugin>mock_components/GenericSystem</plugin>
+    </hardware>
+    -->
     <joint name="left_front_wheel_joint">
       <command_interface name="velocity">
